Commit message: Basically finished

File: larger-arm/urdf/larger-arm.urdf (robot description, URDF)
Before this commit: robot larger-arm, 7 links, 6 joints
Joints:
- joint joint1: limit lower=-3.14 upper=3.14 effort=4000 velocity=100 -> lower=-3.14 upper=3.14 effort=400 velocity=100
- joint joint2: limit lower=-3.14 upper=3.14 effort=4000 velocity=100 -> lower=-3.14 upper=3.14 effort=400 velocity=100
- joint joint3: limit lower=-3.14 upper=3.14 effort=4000 velocity=100 -> lower=-3.14 upper=3.14 effort=400 velocity=100
- joint joint4: limit lower=-3.14 upper=3.14 effort=4000 velocity=100 -> lower=-3.14 upper=3.14 effort=400 velocity=100
